File: PCBs/Power1/Power_grad.sch (EAGLE design)
At the start: 21 parts

Commit message: Power modify
Parts:
- removed 12V_B, 5V_B, GND_B, GND_B_: (no value), ALL:PINHD-1X1
- removed 5V_DRIVER: (no value), ALL:CON_PTR_2
- added U$3: DC-DC-STEP-DOWN-LM2596, ALL:DC-DC-STEP-DOWN-LM2596
- FUSE_ESP, FUSE_ESP1, FUSE_ESP2: value FUSEBLANK_5X20MM -> (none); device fuse:FUSEBLANK_5X20MM -> ALL:FUSE_HOLDER
Connections:
- net 12V: now also U$3.IN+; no longer 12V_B.1, 5V_DRIVERG$1.KL
- net 5V: now also U$3.OUT+; no longer 5V_B.1
- net GND: now also U$3.IN-, U$3.OUT-; no longer 5V_DRIVERG$2.KL, GND_B.1, GND_B_.1
Other:
- moved on the sheet: SWITCH, U$1, U$2
