File: PCBs/Power1/Power_grad2.brd (EAGLE design)
At the start: 112.7 x 101.6 mm, 17 parts

Commit message: PID v1.0
Parts:
- removed 5V_DRIVER1: (no value), ALL:AK300/2
- removed SWITCH: HB9500-9.5-2P, HB9500-9.5-2P:SHDR2W140P0X950_1X2_2055X1800X
- added ALGO, MOTOR, SENSOR: (no value), ALL:DS-01
- added CYTRON: (no value), ALL:AK300/2
- moved U$2 160.1 mm to (80.6, 26.3), turned to 270 degrees
- moved U$1 129.6 mm to (82.2, 33.7)
- moved ALG 123.6 mm to (79.8, 53.2), turned to 270 degrees
- moved SEN 109.4 mm to (79.2, 44.0), turned to 270 degrees
- moved MOT 98.0 mm to (79.8, 61.9), turned to 270 degrees
- moved FUSE_ESP2 92.3 mm to (65.4, 53.2), turned to 90 degrees
- moved U$3 89.1 mm to (53.4, 19.2)
- moved FUSE_ESP1 82.6 mm to (30.5, 52.9), turned to 90 degrees
- moved GND3 78.8 mm to (12.7, 63.5), turned to 90 degrees
- moved FUSE_ESP 73.9 mm to (48.5, 53.5), turned to 90 degrees
- moved 5V_SPARE 72.8 mm to (20.8, 54.7), turned to 270 degrees
- moved GND 72.7 mm to (13.0, 76.5), turned to 90 degrees
- moved GND2 72.2 mm to (12.8, 54.2), turned to 90 degrees
- moved GND1 67.0 mm to (12.7, 44.6), turned to 90 degrees
- moved SUPPLY 45.1 mm to (10.7, 12.0)
Connections:
- removed net 12V_IN: SUPPLY.1, SWITCH.1
- new net N$2: FUSE_ESP1.2, SENSOR.2
- new net N$3: FUSE_ESP.2, MOTOR.2
- new net N$4: ALGO.2, FUSE_ESP2.2
- net 12V: now also CYTRON.1, SUPPLY.1; no longer 5V_DRIVER1.1, SWITCH.2
- net 5V: now also ALGO.1, MOTOR.1, SENSOR.1; no longer FUSE_ESP.2, FUSE_ESP1.2, FUSE_ESP2.2
- net GND: now also CYTRON.2; no longer 5V_DRIVER1.2
Routing:
- net GND: track 0.00 -> 409.7 mm
- net 12V: track 0.00 -> 239.9 mm
- net 5V: track 0.00 -> 152.1 mm
- net SEN: track 0.00 -> 55.1 mm
- net MOT: track 0.00 -> 47.7 mm
- net ALG: track 0.00 -> 27.1 mm
- net N$2: track 0.00 -> 8.45 mm
- net N$3: track 0.00 -> 6.82 mm
- net N$4: track 0.00 -> 6.82 mm
- net N$1: track 0.00 -> 3.88 mm
Other:
- board size 112.7 x 101.6 mm -> 96 x 95.5 mm
